Commit message: update

File: scout_description/urdf/mini.xacro (robot description, xacro)
@@ -11,7 +11,7 @@
     <xacro:property name="M_PI" value="3.14159"/>
     <!-- Vehicle Geometries -->
-    <xacro:property name="base_x_size" value="0.6200000" />
-    <xacro:property name="base_y_size" value="0.585000" />
-    <xacro:property name="base_z_size" value="0.235000" />
+    <xacro:property name="base_x_size" value="0.514618" />
+    <xacro:property name="base_y_size" value="0.3816" />
+    <xacro:property name="base_z_size" value="0.10357" />
     <xacro:property name="wheelbase" value="0.463951"/>
     <xacro:property name="track" value="0.416503"/>
@@ -20,6 +20,6 @@
     <xacro:property name="wheelbase" value="0.3181"/>
     <xacro:property name="wheel_vertical_offset" value="-0.160000047342231" />-->
-    <xacro:property name="wheel_length" value="0.8e-01" />
-    <xacro:property name="wheel_radius" value="1.600e-01" />
+    <xacro:property name="wheel_length" value="0.08" />
+    <xacro:property name="wheel_radius" value="0.08" />
     <!-- Base link -->
     <link name="base_link">
@@ -27,5 +27,5 @@
             <origin
                     xyz="0 0 0.0"
-                    rpy="1.57 0 1.57" />
+                    rpy="1.57 0 -1.57" />
             <geometry>
                 <mesh filename="package://scout_description/meshes/scout_mini_base_link2.dae" />
@@ -35,8 +35,9 @@
             <origin
                     xyz="0 0 0"
-                    rpy="1.57 0 1.57" />
+                    rpy="0 0 0" />
           <geometry>
-            <mesh
-              filename="package://scout_description/meshes/scout_mini_base_link2.dae" />
+            <!--<mesh
+              filename="package://scout_description/meshes/scout_mini_base_link2.dae" />-->
+              <box size="${base_x_size} ${base_y_size} ${base_z_size}"/>
           </geometry>
         </collision>

File: scout_description/urdf/scout_mini_wheel_1.xacro (robot description, xacro)
@@ -40,7 +40,7 @@
             </visual>-->
             <inertial>
-                <mass value="3" />
+                <mass value="15" />
                 <origin xyz="0 0 0" />
-                <inertia ixx="0.7171" ixy="0" ixz="0" iyy="0.7171" iyz="0" izz="0.1361" />
+                <inertia ixx="0.6171" ixy="0" ixz="0" iyy="0.6171" iyz="0" izz="0.1361" />
                 <!--<inertia ixx="0" ixy="0" ixz="0" iyy="0" iyz="0" izz="0" />-->
             </inertial>
@@ -53,9 +53,10 @@
             <collision>
               <origin
-                xyz="0 0 0"
+                xyz="0 0 0.04"
                 rpy="0 0 0" />
               <geometry>
-                <mesh
-                  filename="package://scout_description/meshes/wheel.dae" />
+                <!--<mesh
+                  filename="package://scout_description/meshes/wheel.dae" />-->
+                  <cylinder length="${wheel_length}" radius="${wheel_radius}" />
               </geometry>
             </collision>

File: scout_description/urdf/scout_mini_wheel_2.xacro (robot description, xacro)
@@ -40,7 +40,7 @@
             </visual>-->
             <inertial>
-                <mass value="3" />
+                <mass value="15" />
                 <origin xyz="0 0 0" />
-                <inertia ixx="0.7171" ixy="0" ixz="0" iyy="0.7171" iyz="0" izz="0.1361" />
+                <inertia ixx="0.6171" ixy="0" ixz="0" iyy="0.6171" iyz="0" izz="0.1361" />
                 <!--<inertia ixx="0" ixy="0" ixz="0" iyy="0" iyz="0" izz="0" />-->
             </inertial>
@@ -53,9 +53,10 @@
             <collision>
               <origin
-                xyz="0 0 0"
+                xyz="0 0 0.04"
                 rpy="0 0 0" />
               <geometry>
-                <mesh
-                  filename="package://scout_description/meshes/wheel.dae" />
+                <!--<mesh
+                  filename="package://scout_description/meshes/wheel.dae" />-->
+                  <cylinder length="${wheel_length}" radius="${wheel_radius}" />
               </geometry>
             </collision>

File: scout_description/urdf/scout_mini_wheel_3.xacro (robot description, xacro)
@@ -40,7 +40,7 @@
             </visual>-->
             <inertial>
-                <mass value="3" />
+                <mass value="15" />
                 <origin xyz="0 0 0" />
-                <inertia ixx="0.7171" ixy="0" ixz="0" iyy="0.7171" iyz="0" izz="0.1361" />
+                <inertia ixx="0.6171" ixy="0" ixz="0" iyy="0.6171" iyz="0" izz="0.1361" />
                 <!--<inertia ixx="0" ixy="0" ixz="0" iyy="0" iyz="0" izz="0" />-->
             </inertial>
@@ -53,9 +53,10 @@
             <collision>
               <origin
-                xyz="0 0 0"
+                xyz="0 0 0.04"
                 rpy="0 0 0" />
               <geometry>
-                <mesh
-                  filename="package://scout_description/meshes/wheel.dae" />
+                <!--<mesh
+                  filename="package://scout_description/meshes/wheel.dae" />-->
+                  <cylinder length="${wheel_length}" radius="${wheel_radius}" />
               </geometry>
             </collision>

File: scout_description/urdf/scout_mini_wheel_4.xacro (robot description, xacro)
@@ -40,7 +40,7 @@
         </visual>-->
         <inertial>
-            <mass value="3" />
+            <mass value="15" />
             <origin xyz="0 0 0" />
-            <inertia ixx="0.7171" ixy="0" ixz="0" iyy="0.7171" iyz="0" izz="0.1361" />
+            <inertia ixx="0.6171" ixy="0" ixz="0" iyy="0.6171" iyz="0" izz="0.1361" />
             <!--<inertia ixx="0" ixy="0" ixz="0" iyy="0" iyz="0" izz="0" />-->
         </inertial>
@@ -53,9 +53,10 @@
             <collision>
               <origin
-                xyz="0 0 0"
+                xyz="0 0 0.04"
                 rpy="0 0 0" />
               <geometry>
-                <mesh
-                  filename="package://scout_description/meshes/wheel.dae" />
+                <!--<mesh
+                  filename="package://scout_description/meshes/wheel.dae" />-->
+                  <cylinder length="${wheel_length}" radius="${wheel_radius}" />
               </geometry>
             </collision>

Commit message: add rtabmap navigation

File: scout_description/urdf/mini.xacro (robot description, xacro)
@@ -8,4 +8,5 @@
     <xacro:include filename="$(find scout_description)/urdf/scout_mini_wheel_3.xacro" />
     <xacro:include filename="$(find scout_description)/urdf/scout_mini_wheel_4.xacro" />
+    <xacro:include filename="$(find scout_description)/urdf/scout_mini.gazebo"/>
     <!-- Variables -->
     <xacro:property name="M_PI" value="3.14159"/>
@@ -27,5 +28,5 @@
             <origin
                     xyz="0 0 0.0"
-                    rpy="1.57 0 -1.57" />
+                    rpy="1.57 0.0 -1.57" />
             <geometry>
                 <mesh filename="package://scout_description/meshes/scout_mini_base_link2.dae" />
@@ -59,4 +60,32 @@
         <parent link="base_link" />
         <child link="inertial_link" />
+    </joint>
+    <link name="t265_link">
+        <visual>
+            <origin xyz="0.0 0.0 0.0" />
+            <geometry>
+                <cylinder length="0.03" radius="0.02" />
+            </geometry>
+            <material name="red" />
+        </visual>
+    </link>
+    <joint name="t265_joint" type="fixed">
+        <parent link="base_link" />
+        <child link="t265_link" />
+        <origin xyz="0.32 0.0 0.18" rpy="0 0.2 0" />
+    </joint>
+    <link name="l515_link">
+        <visual>
+            <origin xyz="0.0 0.0 0.0" />
+            <geometry>
+                <cylinder length="0.03" radius="0.02" />
+            </geometry>
+            <material name="red" />
+        </visual>
+    </link>
+    <joint name="l515_joint" type="fixed">
+        <parent link="base_link" />
+        <child link="l515_link" />
+        <origin xyz="0.32 0.0 0.18" rpy="0 0 0" />
     </joint>
     <!-- For testing, hang the robot up in the air -->
@@ -98,3 +127,30 @@
     <!-- Gazebo definitions  -->
     <xacro:include filename="$(find scout_description)/urdf/scout_mini.gazebo" />
+    <joint name="scan_joint" type="fixed">
+      <parent link="base_link"/>
+      <child link="base_scan"/>
+      <origin xyz="-0.000 0.000 0.072" rpy="0 0 0"/>
+    </joint>
+    <link name="base_scan">
+      <visual>
+        <origin xyz="0 0 0.0" rpy="0 0 0"/>
+        <geometry>
+          <mesh filename="package://scout_description/meshes/lds.stl" scale="0.001 0.001 0.001"/>
+        </geometry>
+        <material name="dark"/>
+      </visual>
+      <collision>
+        <origin xyz="0.015 0 -0.0065" rpy="0 0 0"/>
+        <geometry>
+          <cylinder length="0.0315" radius="0.055"/>
+        </geometry>
+      </collision>
+      <inertial>
+        <mass value="0.114" />
+        <origin xyz="0 0 0" />
+        <inertia ixx="0.1" ixy="0.0" ixz="0.0"
+               iyy="0.1" iyz="0.0"
+               izz="0.1" />
+      </inertial>
+  </link>
 </robot>

File: scout_description/urdf/scout_mini.urdf (robot description, URDF)
Before this commit: robot scout_mini, 6 links, 5 joints
Links:
- added link t265_link; visual cylinder length=0.03 radius=0.02
Joints:
- added joint t265_joint: type fixed, parent base_link, child t265_link, origin xyz=0.32 0.0 0.18 rpy=0 0 0

Commit message: update code

File: scout_description/urdf/mini.xacro (robot description, xacro)
@@ -27,5 +27,5 @@
         <visual>
             <origin
-                    xyz="0 0 0.0"
+                    xyz="0 0 -0.30"
                     rpy="1.57 0.0 -1.57" />
             <geometry>
@@ -62,11 +62,10 @@
     </joint>
     <link name="t265_link">
-        <visual>
-            <origin xyz="0.0 0.0 0.0" />
+        <!-- <visual>
+            <origin xyz="0.0 0.0 0.3" />
             <geometry>
-                <cylinder length="0.03" radius="0.02" />
+                <mesh filename="package://scout_description/meshes/l515.dae" />
             </geometry>
-            <material name="red" />
-        </visual>
+        </visual> -->
     </link>
     <joint name="t265_joint" type="fixed">
@@ -76,11 +75,11 @@
     </joint>
     <link name="l515_link">
-        <visual>
-            <origin xyz="0.0 0.0 0.0" />
+        <!-- <visual>
+            <origin xyz="0.0 0.0 0.3" />
             <geometry>
                 <cylinder length="0.03" radius="0.02" />
             </geometry>
             <material name="red" />
-        </visual>
+        </visual> -->
     </link>
     <joint name="l515_joint" type="fixed">
@@ -103,5 +102,5 @@
             xyz="0 0 0"
             rpy="0 0 0" />-->
-        <origin xyz="${wheelbase/2} ${track/2} ${wheel_vertical_offset}" rpy="-1.57 0 0" />
+        <origin xyz="${wheelbase/2} ${track/2} ${wheel_vertical_offset-0.3}" rpy="-1.57 0 0" />
     </xacro:scout_mini_wheel_1>
     <xacro:scout_mini_wheel_2 wheel_prefix="rear_left">
@@ -109,5 +108,5 @@
             xyz="0 0 0"
             rpy="0 0 0" />-->
-        <origin xyz="${-wheelbase/2} ${track/2} ${wheel_vertical_offset}" rpy="-1.57 0 0" />
+        <origin xyz="${-wheelbase/2} ${track/2} ${wheel_vertical_offset-0.3}" rpy="-1.57 0 0" />
     </xacro:scout_mini_wheel_2>
     <xacro:scout_mini_wheel_3 wheel_prefix="front_right">
@@ -115,5 +114,5 @@
             xyz="0 0 0"
             rpy="0 0 0" />-->
-        <origin xyz="${wheelbase/2} ${-track/2} ${wheel_vertical_offset+0.001}" rpy="1.57 0 0" />
+        <origin xyz="${wheelbase/2} ${-track/2} ${wheel_vertical_offset+0.001-0.3}" rpy="1.57 0 0" />
     </xacro:scout_mini_wheel_3>
     <xacro:scout_mini_wheel_4 wheel_prefix="rear_right">
@@ -121,5 +120,5 @@
            xyz="0 0 0"
            rpy="0 0 0" />-->
-        <origin xyz="${-wheelbase/2} ${-track/2} ${wheel_vertical_offset+0.001}" rpy="1.57 0 0" />
+        <origin xyz="${-wheelbase/2} ${-track/2} ${wheel_vertical_offset+0.001-0.3}" rpy="1.57 0 0" />
     </xacro:scout_mini_wheel_4>
     <!-- Additional definitions -->
@@ -127,5 +126,5 @@
     <!-- Gazebo definitions  -->
     <xacro:include filename="$(find scout_description)/urdf/scout_mini.gazebo" />
-    <joint name="scan_joint" type="fixed">
+    <!-- <joint name="scan_joint" type="fixed">
       <parent link="base_link"/>
       <child link="base_scan"/>
@@ -153,4 +152,4 @@
                izz="0.1" />
       </inertial>
-  </link>
+  </link> -->
 </robot>
